Commit message: 更新配置文件

File: my_sensor_kit_description/urdf/sensor_kit.xacro (robot description, xacro)
@@ -20,4 +20,20 @@
     <xacro:property name="calibration" value="${xacro.load_yaml('$(arg config_dir)/sensor_kit_calibration.yaml')}"/>
     <!-- lidar -->
+    <xacro:property name="robosense_helios" value="robosense_helios"/>
+    <link name="${robosense_helios}_link">
+      <origin rpy="0 0 0" xyz="0 0 0"/>
+    </link>
+    <joint name="${robosense_helios}_joint" type="fixed">
+      <origin
+        xyz="${calibration['sensor_kit_base_link']['robosense_helios_link']['x']}
+             ${calibration['sensor_kit_base_link']['robosense_helios_link']['y']}
+             ${calibration['sensor_kit_base_link']['robosense_helios_link']['z']}"
+        rpy="${calibration['sensor_kit_base_link']['robosense_helios_link']['roll']}
+             ${calibration['sensor_kit_base_link']['robosense_helios_link']['pitch']}
+             ${calibration['sensor_kit_base_link']['robosense_helios_link']['yaw']}"
+      />
+      <parent link="${sensor_kit_base_link}"/>
+      <child link="${robosense_helios}_link"/>
+    </joint>
     <!-- <xacro:VLS-128 parent="sensor_kit_base_link" name="velodyne_top" topic="/points_raw" hz="10" samples="220" gpu="$(arg gpu)">
       <origin
